File: electronics/RPI4Soar_V1.brd (EAGLE design)
At the start: 93.7 x 57.1 mm, 26 parts, among them IC1 MAX3232CPE, J1 RASPBERRYPI-40-PIN-GPIO_PTH_R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, J2 FEMALE 2x3, J3 J3, J4 J4, J6 J6, J7 J7

Commit message: add RPI4Soar BOM
Parts:
- F1: value 72V/0.25A -> 30V/3.5A
Changed lines of the file:
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@@
 <attribute name="VALUE" x="23.876" y="15.367" size="1.27" layer="27" ratio="10" rot="R270"/>
 </element>
-<element name="F1" library="SparkFun-Fuses" package="PTH" value="72V/0.25A" x="26.67" y="27.305" smashed="yes" rot="R90">
+<element name="F1" library="SparkFun-Fuses" package="PTH" value="30V/3.5A" x="26.67" y="27.305" smashed="yes" rot="R90">
 <attribute name="NAME" x="24.892" y="27.305" size="0.6096" layer="25" font="vector" ratio="20" rot="R90" align="bottom-center"/>
 <attribute name="PROD_ID" value="RES-08490" x="26.67" y="27.305" size="1.778" layer="27" rot="R90" display="off"/>
