File: electronics/RPI4Soar_V1.sch (EAGLE design)
At the start: 26 parts, among them IC1 MAX3232CPE, J1 RASPBERRYPI-40-PIN-GPIO_PTH_R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, J2 FEMALE 2x3, J3 J3, J4 J4, J6 J6, J7 J7

Commit message: add RPI4Soar BOM
Parts:
- F1: value 72V/0.25A -> 30V/3.5A
Changed lines of the file:
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@@
 <part name="J2" library="SparkFun-Connectors" deviceset="CONN_03X2" device="FEMALE" value="FEMALE 2x3"/>
 <part name="D1" library="adafruit" deviceset="1N4004" device=""/>
-<part name="F1" library="SparkFun-Fuses" deviceset="PPTC" device="_PTH" value="72V/0.25A"/>
+<part name="F1" library="SparkFun-Fuses" deviceset="PPTC" device="_PTH" value="30V/3.5A"/>
 <part name="J4" library="SparkFun-Connectors" deviceset="CONN_03" device="" value="J4"/>
 <part name="R1" library="SparkFun-Resistors" deviceset="RESISTOR" device="AXIAL-0.3" value=" "/>
